Commit message: added xacro

File: my_pkg/urdf/common_props.xacro (robot description, xacro)
@@ -2,8 +2,8 @@
   <robot xmlns:xacro="http://www.ros.org/wiki/xacro">
     <material name="blue">
-        <color rgba="0.5 1 0.5 1" />
+        <color rgba="1 0.5 0.5 1" />
     </material>
     <material name="grey">
-        <color rgba="0.5 1.0 1.0 1" />
+        <color rgba="0.5 0.5 1.0 1" />
     </material>
   </robot>

File: my_pkg/urdf/my_robot.urdf.xacro (robot description, xacro)
@@ -1,109 +1,5 @@
 <?xml version="1.0"?>
   <robot name="my_robot" xmlns:xacro="http://www.ros.org/wiki/xacro">
-    <xacro:include filename="common_prop.xacro"/>
-    <xacro:property name="base_len" value="1.0"/>
-      <link name="world" />
-      <link name="base_link">
-          <visual>
-              <geometry>
-                  <box size="${base_len} 0.4 0.2" />
-              </geometry>
-              <origin xyz="-3 -2 0.1" rpy="0 0 0" />
-              <material name="blue" />
-          </visual>
-      </link>
-        <joint name="base_world" type="fixed">
-            <parent link="world" />
-            <child link="base_link" />
-            <origin xyz="0 0 0.1" rpy="0 0 0"/>
-        </joint>
-    <link name="right_wheel_link">
-          <visual>
-              <geometry>
-                  <cylinder radius="0.1" length="0.05" />
-              </geometry>
-              <origin xyz="0 0 0" rpy="${pi / 2.0} 0 0" />
-              <material name="grey" />
-          </visual>
-    </link>
-    <xacro:macro name="macro_wheel_link" params="prefix">
-        <link name="${prefix}_wheel_link">
-            <visual>
-                <geometry>
-                    <cylinder radius="0.1" length="0.05" />
-                </geometry>
-                <origin xyz="0 0 0" rpy="${pi / 2.0} 1.0 1.0" />
-                <material name="grey" />
-            </visual>
-      </link>
-    </xacro:macro>
-    <xacro:macro_wheel_link prefix="back"/>
-    <joint name="base_back_wheel_joint" type="continuous">
-        <parent link="base_link"/>
-        <child link="back_wheel_link"/>
-        <origin xyz="${-base_len / 4.0} -0.225 0" rpy="0 0 0" />
-        <axis xyz="0 1 0" />
-      </joint>
-    <joint name="base_right_wheel_joint" type="continuous">
-      <parent link="base_link"/>
-      <child link="right_wheel_link"/>
-      <origin xyz="${-base_len / 4.0} -0.225 0" rpy="0 0 0" />
-      <axis xyz="0 1 0" />
-    </joint>
-    <link name="left_wheel_link">
-        <visual>
-            <geometry>
-                <cylinder radius="0.1" length="0.05" />
-            </geometry>
-            <origin xyz="0 0 0" rpy="${pi / 2.0} 0 0" />
-            <material name="grey" />
-        </visual>
-    </link>
-    <joint name="base_left_wheel_joint" type="continuous">
-        <parent link="base_link" />
-        <child link="left_wheel_link" />
-        <origin xyz="-0.15 0.225 0" rpy="0 0 0" />
-        <axis xyz="0 1 0" />
-    </joint>
-    <link name="caster_wheel_link">
-        <visual>
-            <geometry>
-                <sphere radius="0.05" />
-            </geometry>
-            <origin xyz="0 0 0" rpy="0 0 0" />
-            <material name="grey" />
-        </visual>
-    </link>
-    <joint name="base_caster_wheel_joint" type="fixed">
-        <parent link="base_link" />
-        <child link="caster_wheel_link" />
-        <origin xyz="${base_len / 3.0} 0 -0.05" rpy="0 0 0" />
-    </joint>
-    <link name="new_link">
-        <visual>
-            <geometry>
-                <sphere radius="0.5"/>
-            </geometry>
-        </visual>
-    </link>
-    <joint name="new_world" type="fixed">
-        <parent link="world" />
-        <child link="new_link" />
-        <origin xyz="3 2 -0.05" rpy="0 0 0" />
-    </joint>
-    <link name="new_wheel_link">
-        <visual>
-            <geometry>
-                <cylinder radius="0.1" length="0.01" />
-            </geometry>
-            <origin xyz="0 0 0" rpy="${pi / 2.0} 0 0" />
-            <material name="grey" />
-        </visual>
-    </link>
-    <joint name="new_left_wheel_joint" type="continuous">
-        <parent link="new_link" />
-        <child link="new_wheel_link" />
-        <origin xyz="-0.15 0.225 0" rpy="0 0 0" />
-        <axis xyz="0 1 0" />
-    </joint>
+    <xacro:include filename="common_props.xacro"/>
+    <xacro:include filename="mobile_bot.xacro"/>
   </robot>

Commit message: added gz launch and fixed colors

File: my_pkg/urdf/common_props.xacro (robot description, xacro)
@@ -7,3 +7,30 @@
         <color rgba="0.5 0.5 1.0 1" />
     </material>
+    <xacro:macro name="box_inertia" params="m l w h xyz rpy" >
+      <inertial>
+        <origin xyz="${xyz}" rpy="${rpy}"/>
+        <mass value="${m}"/>
+        <inertia ixx="${(m/12)*(h*h + l*l)}" ixy="0" ixz="0"
+          iyy="${(m/12) * (w*w + l*l)}" iyz="0.0"
+          izz="${(m/12) * (w*w + h*h)}"/>
+      </inertial>
+    </xacro:macro>
+    <xacro:macro name="cylinder_inertia" params="m r h xyz rpy" >
+      <inertial>
+        <origin xyz="${xyz}" rpy="${rpy}"/>
+        <mass value="${m}"/>
+        <inertia ixx="${(m/12)*(3*r*r + h*h)}" ixy="0" ixz="0"
+          iyy="${(m/12)*(3*r*r + h*h)}" iyz="0.0"
+          izz="${(m/2) * (r*r)}"/>
+      </inertial>
+    </xacro:macro>
+    <xacro:macro name="sphere_inertia" params="m r xyz rpy" >
+      <inertial>
+        <origin xyz="${xyz}" rpy="${rpy}"/>
+        <mass value="${m}"/>
+        <inertia ixx="${(2/5)* m * r * r}" ixy="0" ixz="0"
+          iyy="${(2/5)* m * r * r}" iyz="0.0"
+          izz="${(2/5)* m * r * r}"/>
+      </inertial>
+    </xacro:macro>
   </robot>

File: my_pkg/urdf/mobile_bot.xacro (robot description, xacro)
@@ -4,6 +4,6 @@
     <xacro:property name="base_w" value="0.4"/>
     <xacro:property name="base_h" value="0.2"/>
-    <xacro:property name="wheel_rad" value="0.2"/>
-    <xacro:property name="wheel_len" value="0.01"/>
+    <xacro:property name="wheel_rad" value="0.1"/>
+    <xacro:property name="wheel_len" value="0.05"/>
       <link name="world" />
       <link name="base_link">
@@ -15,15 +15,12 @@
               <material name="blue" />
           </visual>
-          <inertial>
-            <origin xyz="0.0 0.0 0.0" rpy="0.0 0.0 0.0"/>
-            <mass value="0.0"/>
-            <inertia ixx="0.0" ixy="0.0" ixz="0.0" iyy="0.0" iyz="0.0" izz="0.0"/>
-          </inertial>
           <collision>
             <geometry>
-                <box size="1.0 0.4 0.2" />
+                <box size="${base_len} ${base_w} ${base_h}" />
             </geometry>
-            <origin xyz="-3 -2 0.1" rpy="0 0 0" />
+            <origin xyz="0 0 ${base_h / 2.0}" rpy="0 0 0" />
           </collision>
+          <xacro:box_inertia m="5.0" l="${2*base_len}" w="${2*base_w}" h="${2*base_h}"
+            xyz="0 0 ${base_h / 2.0}" rpy="0 0 0"/>
         </link>
         <joint name="base_world" type="fixed">
@@ -32,46 +29,31 @@
             <origin xyz="0 0 0.1" rpy="0 0 0"/>
         </joint>
-    <link name="right_wheel_link">
-          <visual>
-              <geometry>
-                  <cylinder radius="${wheel_rad}" length="0.05" />
-              </geometry>
-              <origin xyz="0 0 0" rpy="${pi / 2} 0 0" />
-              <material name="grey" />
-          </visual>
-    </link>
     <xacro:macro name="macro_wheel_link" params="prefix">
         <link name="${prefix}_wheel_link">
             <visual>
                 <geometry>
-                    <cylinder radius="0.1" length="0.05" />
+                    <cylinder radius="${wheel_rad}" length="${wheel_len}" />
                 </geometry>
-                <origin xyz="0 0 0" rpy="1.57 1.0 1.0" />
+                <origin xyz="0 0 0" rpy="${pi / 2.0} 1.0 1.0" />
                 <material name="grey" />
             </visual>
+            <collision>
+                <geometry>
+                    <cylinder radius="${wheel_rad}" length="${wheel_len}" />
+                </geometry>
+                <origin xyz="0 0 0" rpy="${pi / 2.0} 1.0 1.0" />
+            </collision>
+            <xacro:cylinder_inertia m="1.0" r="${wheel_rad}" h="${wheel_len}"
+                xyz="0 0 0" rpy="${pi / 2.0} 1.0 1.0" />
       </link>
     </xacro:macro>
-    <xacro:macro_wheel_link prefix="back"/>
-    <joint name="base_back_wheel_joint" type="continuous">
+    <xacro:macro_wheel_link prefix="right"/>
+    <xacro:macro_wheel_link prefix="left"/>
+    <joint name="base_right_wheel_joint" type="continuous">
         <parent link="base_link"/>
-        <child link="back_wheel_link"/>
-        <origin xyz="0.25 -0.225 0" rpy="0 0 0" />
+        <child link="right_wheel_link"/>
+        <origin xyz="${-base_len / 4.0} ${-(base_w + wheel_len) / 2.0} 0" rpy="0 0 0" />
         <axis xyz="0 1 0" />
       </joint>
-    <joint name="base_right_wheel_joint" type="continuous">
-      <parent link="base_link"/>
-      <child link="right_wheel_link"/>
-      <origin xyz="${-base_len / 4.0} ${-(base_w + wheel_len) / 2.0} 0" rpy="0 0 0" />
-      <axis xyz="0 1 0" />
-    </joint>
-    <link name="left_wheel_link">
-        <visual>
-            <geometry>
-                <cylinder radius="${wheel_rad}" length="0.05" />
-            </geometry>
-            <origin xyz="0 0 0" rpy="1.57 0 0" />
-            <material name="grey" />
-        </visual>
-    </link>
     <joint name="base_left_wheel_joint" type="continuous">
         <parent link="base_link" />
@@ -88,36 +70,16 @@
             <material name="grey" />
         </visual>
+        <collision>
+            <geometry>
+                <sphere radius="${wheel_rad / 2.0}" />
+            </geometry>
+            <origin xyz="0 0 0" rpy="0 0 0" />
+        </collision>
+        <xacro:sphere_inertia m="0.5" r="${wheel_rad / 2.0}" xyz="0 0 0" rpy="0 0 0"/>
     </link>
     <joint name="base_caster_wheel_joint" type="fixed">
         <parent link="base_link" />
         <child link="caster_wheel_link" />
-        <origin xyz="0.5 0 ${-wheel_rad / 2.0}" rpy="0 0 0" />
+        <origin xyz="${base_len / 3.0} 0 ${-wheel_rad / 2.0}" rpy="0 0 0" />
     </joint>
-    <!-- <link name="new_link">
-        <visual>
-            <geometry>
-                <sphere radius="0.5"/>
-            </geometry>
-        </visual>
-    </link> -->
-    <!-- <joint name="new_world" type="fixed">
-        <parent link="world" />
-        <child link="new_link" />
-        <origin xyz="3 2 -0.05" rpy="0 0 0" />
-    </joint> -->
-    <!-- <link name="new_wheel_link">
-        <visual>
-            <geometry>
-                <cylinder radius="0.1" length="0.01" />
-            </geometry>
-            <origin xyz="0 0 0" rpy="1.57 0 0" />
-            <material name="grey" />
-        </visual>
-    </link> -->
-    <!-- <joint name="new_left_wheel_joint" type="continuous">
-        <parent link="new_link" />
-        <child link="new_wheel_link" />
-        <origin xyz="-0.15 0.225 0" rpy="0 0 0" />
-        <axis xyz="0 1 0" />
-    </joint>  -->
   </robot>

File: my_pkg/urdf/my_robot.urdf.xacro (robot description, xacro)
@@ -3,3 +3,4 @@
     <xacro:include filename="common_props.xacro"/>
     <xacro:include filename="mobile_bot.xacro"/>
+    <xacro:include filename="mobile_bot_gazebo.xacro"/>
   </robot>

Commit message: added robot arm

File: my_pkg/urdf/common_props.xacro (robot description, xacro)
@@ -6,4 +6,10 @@
     <material name="grey">
         <color rgba="0.5 0.5 1.0 1" />
+    </material>
+    <material name="yellow">
+      <color rgba="0.5 0.5 1.0 1" />
+    </material>
+    <material name="orange">
+      <color rgba="1.0 0.5 0 1" />
     </material>
     <xacro:macro name="box_inertia" params="m l w h xyz rpy" >

File: my_pkg/urdf/mobile_bot.xacro (robot description, xacro)
@@ -35,5 +35,5 @@
                     <cylinder radius="${wheel_rad}" length="${wheel_len}" />
                 </geometry>
-                <origin xyz="0 0 0" rpy="${pi / 2.0} 1.0 1.0" />
+                <origin xyz="0 0 0" rpy="${pi / 2.0} 0 0" />
                 <material name="grey" />
             </visual>
@@ -42,5 +42,5 @@
                     <cylinder radius="${wheel_rad}" length="${wheel_len}" />
                 </geometry>
-                <origin xyz="0 0 0" rpy="${pi / 2.0} 1.0 1.0" />
+                <origin xyz="0 0 0" rpy="${pi / 2.0} 0 0" />
             </collision>
             <xacro:cylinder_inertia m="1.0" r="${wheel_rad}" h="${wheel_len}"
@@ -78,5 +78,5 @@
         <xacro:sphere_inertia m="0.5" r="${wheel_rad / 2.0}" xyz="0 0 0" rpy="0 0 0"/>
     </link>
-    <joint name="base_caster_wheel_joint" type="fixed">
+    <joint name="base_caster_wheel_joint" type="continuous">
         <parent link="base_link" />
         <child link="caster_wheel_link" />

File: my_pkg/urdf/mobile_bot_gazebo.xacro (robot description, xacro)
@@ -2,14 +2,38 @@
 <robot xmlns:xacro="http://www.ros.org/wiki/xacro" >
     <gazebo reference="base_link">
+        <material>Gazebo/Red</material>
+    </gazebo>
+    <gazebo reference="right_wheel_link">
         <material>Gazebo/Blue</material>
     </gazebo>
-    <gazebo reference="right_wheel_link">
-        <material>Gazebo/Grey</material>
-    </gazebo>
     <gazebo reference="left_wheel_link">
-        <material>Gazebo/Grey</material>
+        <material>Gazebo/Blue</material>
     </gazebo>
     <gazebo reference="caster_wheel_link">
-        <material>Gazebo/Grey</material>
+        <material>Gazebo/Blue</material>
+    </gazebo>
+    <gazebo>
+        <plugin name="diff_drive_controller" filename="libgazebo_ros_diff_drive.so">
+            <!-- Update rate in Hz -->
+            <update_rate>50</update_rate>
+            <!-- wheels -->
+            <left_joint>base_left_wheel_joint</left_joint>
+            <right_joint>base_right_wheel_joint</right_joint>
+            <!-- kinematics -->
+            <wheel_separation>0.45</wheel_separation>
+            <wheel_diameter>0.2</wheel_diameter>
+            <!-- limits
+            <max_wheel_torque>20</max_wheel_torque>
+            <max_wheel_acceleration>1.0</max_wheel_acceleration> -->
+            <!-- input
+            <command_topic>cmd_vel</command_topic> -->
+            <!-- output -->
+            <publish_odom>true</publish_odom>
+            <publish_odom_tf>true</publish_odom_tf>
+            <publish_wheel_tf>true</publish_wheel_tf>
+            <odometry_topic>odom</odometry_topic>
+            <odometry_frame>odom</odometry_frame>
+            <robot_base_frame>world</robot_base_frame>
+          </plugin>
     </gazebo>
 </robot>

File: my_pkg/urdf/my_robot.urdf.xacro (robot description, xacro)
@@ -4,3 +4,5 @@
     <xacro:include filename="mobile_bot.xacro"/>
     <xacro:include filename="mobile_bot_gazebo.xacro"/>
+    <xacro:include filename="camera.xacro"/>
+    <xacro:include filename="arm.xacro"/>
   </robot>
