Commit message: finished course  https://www.udemy.com/course/ros2-advanced-core-concepts

File: my_pkg/urdf/arm.xacro (robot description, xacro)
@@ -6,5 +6,5 @@
     <xacro:property name="forearm_rad" value="0.02" />
     <xacro:property name="forearm_len" value="0.3" />
-    <link name="world"/>
+    <link name="world_arm"/>
     <link name="arm_base_link">
         <visual>
@@ -15,7 +15,15 @@
         <material name="orange"/>
         </visual>
+        <collision>
+            <geometry>
+                <box size="${arm_base_len} ${arm_base_w}  ${arm_base_h}"/>
+            </geometry>
+            <origin xyz="0 0 ${arm_base_h / 2}" rpy="0 0 0"/>
+        </collision>
+        <xacro:box_inertia m="0.5" l="${2*arm_base_len}" w="${2*arm_base_w}" h="${2*arm_base_h}"
+        xyz="0 0 ${arm_base_h / 2}" rpy="0 0 0"/>
     </link>
-    <joint name="base_world" type="fixed">
-        <parent link="world" />
+    <joint name="base_world_arm" type="fixed">
+        <parent link="world_arm" />
         <child link="arm_base_link" />
         <origin xyz="0 0 0.0" rpy="0 0 0"/>
@@ -29,4 +37,12 @@
             <material name="yellow"/>
         </visual>
+        <collision>
+            <geometry>
+                <cylinder radius="${forearm_rad}" length="${forearm_len}"/>
+            </geometry>
+            <origin xyz="0 0 ${forearm_len / 2}" rpy="0.0 0.0 0.0"/>
+        </collision>
+        <xacro:cylinder_inertia m="0.3" r="${2*forearm_rad}" h="${2*forearm_len}"
+            xyz="0 0 ${forearm_len / 2}" rpy="0.0 0.0 0.0" />
     </link>
     <joint name="forearm_arm_base_joint" type="revolute">
@@ -36,4 +52,5 @@
         <axis xyz="0 1 0"/>
         <limit lower="${-pi/2}" upper="${pi/2}" effort="100" velocity="100"/>
+        <dynamics friction="0.05" damping="0.1"/>
     </joint>
     <link name="hand_link">
@@ -45,4 +62,12 @@
             <material name="Blue"/>
         </visual>
+        <collision>
+            <geometry>
+                <cylinder radius="${forearm_rad}" length="${forearm_len}"/>
+            </geometry>
+            <origin xyz="0 0 ${forearm_len / 2}" rpy="0.0 0.0 0.0"/>
+        </collision>
+        <xacro:cylinder_inertia m="0.3" r="${2*forearm_rad}" h="${2*forearm_len}"
+            xyz="0 0 ${forearm_len / 2}" rpy="0.0 0.0 0.0" />
     </link>
     <joint name="hand_forearm_arm_joint" type="revolute">
@@ -52,4 +77,5 @@
         <axis xyz="0 1 0"/>
         <limit lower="0" upper="${pi/2}" effort="100" velocity="100"/>
+        <dynamics friction="0.05" damping="0.1"/>
     </joint>
 </robot>

File: my_pkg/urdf/my_robot.urdf.xacro (robot description, xacro)
@@ -4,5 +4,11 @@
     <xacro:include filename="mobile_bot.xacro"/>
     <xacro:include filename="mobile_bot_gazebo.xacro"/>
-    <xacro:include filename="camera.xacro"/>
+    <!-- <xacro:include filename="camera.xacro"/> -->
     <xacro:include filename="arm.xacro"/>
+    <xacro:include filename="arm_gazebo.xacro"/>
+    <joint name="mobile_bot_arm_joint" type="fixed">
+      <origin xyz="${base_len / 4} 0 ${base_h}" rpy="0.0 0.0 0.0"/>
+      <parent link="base_link"/>
+      <child link="world_arm"/>
+    </joint>
   </robot>

File: my_pkg/urdf/standalone_arm.urdf.xacro (robot description, xacro)
@@ -3,3 +3,4 @@
     <xacro:include filename="common_props.xacro"/>
     <xacro:include filename="arm.xacro"/>
+    <xacro:include filename="arm_gazebo.xacro" />
 </robot>
