Commit message: added ros control

File: my_pkg/urdf/mobile_bot.xacro (robot description, xacro)
@@ -6,5 +6,5 @@
     <xacro:property name="wheel_rad" value="0.1"/>
     <xacro:property name="wheel_len" value="0.05"/>
-      <link name="world" />
+      <link name="world_mylink" />
       <link name="base_link">
           <visual>
@@ -25,5 +25,5 @@
         </link>
         <joint name="base_world" type="fixed">
-            <parent link="world" />
+            <parent link="world_mylink" />
             <child link="base_link" />
             <origin xyz="0 0 0.1" rpy="0 0 0"/>
@@ -82,4 +82,5 @@
         <child link="caster_wheel_link" />
         <origin xyz="${base_len / 3.0} 0 ${-wheel_rad / 2.0}" rpy="0 0 0" />
+        <dynamics friction="0.1" damping="0.1"/>
     </joint>
   </robot>

File: my_pkg/urdf/my_robot.urdf.xacro (robot description, xacro)
@@ -7,4 +7,5 @@
     <xacro:include filename="arm.xacro"/>
     <xacro:include filename="arm_gazebo.xacro"/>
+    <xacro:include filename="arm_control.xacro"/>
     <joint name="mobile_bot_arm_joint" type="fixed">
       <origin xyz="${base_len / 4} 0 ${base_h}" rpy="0.0 0.0 0.0"/>
